File: WaterDoor_hw/WaterDoor.sch (KiCad schematic (older format))
At the start: 74 parts, among them Q3 IRLMS9303, SW5 SWITCH_H

Commit message: + Main PCB ready for production
Parts:
- removed C29, C31: 1u, CAP_0603, symbol C
- removed C?: 100u, symbol CP
- removed F1: FUSE0R, ~, symbol Fuse0R
- removed XL9: CONN_2, ~, symbol CONN_2
- removed XL? (x9): RJ11, symbol RJ11
- added C3: 10u, CAP_0805, symbol C
- added C5, C6: 1u, CAP_0603, symbol C
- added D1: LED, symbol LED
- added HOLE5, HOLE6: HOLE_METALLED, symbol HOLE_METALLED
- added R1: 2k, symbol R
- added R10, R13, R14, R15, R16, R17, R18, R6, R7, R9: 1k, RES_0603, symbol R
- added XL18, XL19, XL20, XL21, XL22, XL23, XL24, XL25, XL26: RJ11, symbol RJ11
- added XL9: BARREL_SOCKET, symbol BARREL_SOCKET
- gave numbers to parts that had none: 27
Connections:
- net +3.3V: now also XL11.2, XL12.2, XL13.2, XL14.2, XL15.2, XL4.2, XL5.2, XL6.2, XL7.2, XL8.2, C6.1
- net +5V: now also C3.2, C5.1; no longer XL11.2, XL12.2, XL13.2, XL14.2, XL15.2, XL4.2, XL5.2, XL6.2, XL7.2, XL8.2
- net GND: now also XL10.1 (P1), XL17.5, C3.1, C5.2, C6.2, D1.C, HOLE5.H, HOLE6.H, XL18.4, XL18.5, XL18.H (GND), XL19.4, XL19.5, XL19.H (GND), XL20.4, XL20.5, XL20.H (GND), XL21.4, XL21.5, XL21.H (GND), XL22.4, XL22.5, XL22.H (GND), XL23.4, XL23.5, XL23.H (GND), XL24.4, XL24.5, XL24.H (GND), XL25.4, XL25.5, XL25.H (GND), XL26.4, XL26.5, XL26.H (GND), XL9.GND; no longer XL10.2 (PM)
- net LEDS_OUT: now also XL18.3, XL19.3, XL20.3, XL21.3, XL22.3, XL23.3, XL24.3, XL25.3, XL26.3
- net OUT_12V: now also XL10.2 (PM); no longer XL10.1 (P1)
- net SNS1: now also R10.1; no longer DD1.40 (PB4/JTRST/T3C1/MISO1)
- net SNS10: now also R18.1; no longer DD1.21 (PB10/SCL2/TX3/T2C3)
- net SNS2: now also R13.1; no longer DD1.41 (PB5/T3C2/MOSI1)
- net SNS3: now also R6.1; no longer DD1.18 (PB0/T3C3/ADC8)
- net SNS4: now also R7.1; no longer DD1.19 (PB1/T3C4/ADC9)
- net SNS5: now also R14.1; no longer DD1.42 (PB6/SCL1/T4C1/TX1)
- net SNS6: now also R15.1; no longer DD1.43 (PB7/SDA1/T4C2/RX1)
- net SNS7: now also R16.1; no longer DD1.45 (PB8/SCL1/T4C3/T10C1)
- net SNS8: now also R17.1; no longer DD1.46 (PB9/SDA1/T4C4/T11C1)
- net SNS9: now also R9.1; no longer DD1.39 (PB3/JTDO/T2C2/SCK1)
- net +12V: now reaches SW5.2
- net +12V: now also C19.1, C20.1, C21.1, C22.1, DA1.5 (Vcc), DA1.6 (Vcc), DA1.7 (Vcc), DA1.8 (Vcc), DA2.1 (Vin_A), DA2.2 (EN), DA2.6 (Vin_SW), R1.1
- removed net +BATT: C19.1, C20.1, C21.1, C22.1, DA1.5 (Vcc), DA1.6 (Vcc), DA1.7 (Vcc), DA1.8 (Vcc), DA2.1 (Vin_A), DA2.2 (EN), DA2.6 (Vin_SW), SW5.1
- new net: D1.A, R1.2
- new net PWR_IN: SW5.1, XL9.PWR
- new net SNS10R: DD1.21 (PB10/SCL2/TX3/T2C3), R18.2
- new net SNS1R: DD1.40 (PB4/JTRST/T3C1/MISO1), R10.2
- new net SNS2R: DD1.41 (PB5/T3C2/MOSI1), R13.2
- new net SNS3R: DD1.18 (PB0/T3C3/ADC8), R6.2
- new net SNS4R: DD1.19 (PB1/T3C4/ADC9), R7.2
- new net SNS5R: DD1.42 (PB6/SCL1/T4C1/TX1), R14.2
- new net SNS6R: DD1.43 (PB7/SDA1/T4C2/RX1), R15.2
- new net SNS7R: DD1.45 (PB8/SCL1/T4C3/T10C1), R16.2
- new net SNS8R: DD1.46 (PB9/SDA1/T4C4/T11C1), R17.2
- new net SNS9R: DD1.39 (PB3/JTDO/T2C2/SCK1), R9.2
- no-connect marks 76 -> 82
Other:
- note added: "10...15V -> 4.8V for IR LEDs"
- note added: "3.3V power regulator for MCU and IR sensors"
- note added: "USB to UART"
- note removed: "10...15V -> 4.8V"
- note removed: "3.3V 150mA power regulator"
- note removed: "Solder if no need in BUCK"
- moved on the sheet: C1, C12, C13, C14, C15, C16, C18, C19, C2, C20, C21, C22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
